File: BPS-Fan.kicad_pcb (KiCad board)
At the start: 2 copper layers, 57.3 x 82.1 mm, 37 parts, among them J1 LDRBRDConn, J10 FAN9, J11 FAN10, J12 FAN11, J13 FAN12, J2 FAN1, J3 FAN2, J4 FAN3, J5 FAN4, J6 FAN5, J7 FAN6, J8 FAN7, J9 FAN8, Q1 BUK9M23-80E, Q2 BUK9M23-80E, Q3 BUK9M23-80E, Q4 BUK9M23-80E

Commit message: fan go brrr
Parts:
- removed D1, D2, D3, D4: V2F22HM, UTSVT_Passive:V2F22HM
- removed J10: FAN9, UTSVT_Connectors:Molex_MicroFit3.0_1x2xP3.00mm_PolarizingPeg_Vertical
- removed J11: FAN10, UTSVT_Connectors:Molex_MicroFit3.0_1x2xP3.00mm_PolarizingPeg_Vertical
- removed J12: FAN11, UTSVT_Connectors:Molex_MicroFit3.0_1x2xP3.00mm_PolarizingPeg_Vertical
- removed J13: FAN12, UTSVT_Connectors:Molex_MicroFit3.0_1x2xP3.00mm_PolarizingPeg_Vertical
- removed J6: FAN5, UTSVT_Connectors:Molex_MicroFit3.0_1x2xP3.00mm_PolarizingPeg_Vertical
- removed J7: FAN6, UTSVT_Connectors:Molex_MicroFit3.0_1x2xP3.00mm_PolarizingPeg_Vertical
- removed J8: FAN7, UTSVT_Connectors:Molex_MicroFit3.0_1x2xP3.00mm_PolarizingPeg_Vertical
- removed J9: FAN8, UTSVT_Connectors:Molex_MicroFit3.0_1x2xP3.00mm_PolarizingPeg_Vertical
- removed PowerLED: STATUS, LED_SMD:LED_0805_2012Metric
- removed Q3: BUK9M23-80E, Package_TO_SOT_SMD:LFPAK33
- removed R4, R8: 100k, Resistor_SMD:R_0805_2012Metric
- added LED1: STATUS, LED_SMD:LED_0805_2012Metric, F.Cu at (85.6, 85.7)
- added Q5: BUK9M23-80E, Package_TO_SOT_SMD:LFPAK33, F.Cu at (123.6, 83.5)
- added R10: 100k, Resistor_SMD:R_0805_2012Metric, F.Cu at (124.5, 87.7)
- added R11: 100k, Resistor_SMD:R_0805_2012Metric, F.Cu at (122.3, 87.7)
- J2: value FAN1 -> FAN7
- J3: value FAN2 -> FAN7
- J4: value FAN3 -> FAN7
- J5: value FAN4 -> FAN7
- LOGO1, LOGO2: moved to F.Cu
- moved R1 89.0 mm to (90.0, 85.7), turned to 0 degrees
- moved H3 84.4 mm to (117.7, 97.5)
- moved LOGO2 68.4 mm to (92.3, 80.5), turned to 0 degrees
- moved H2 64.8 mm to (153.9, 61.7)
- moved LOGO1 48.7 mm to (93.2, 63.8), turned to 0 degrees
- moved J4 45.6 mm to (153.5, 69.4), turned to -90 degrees
- moved R5 40.2 mm to (147.3, 84.1), turned to -90 degrees
- moved J5 35.3 mm to (117.9, 87.7), turned to 90 degrees
- moved J1 34.0 mm to (139.3, 79.9)
- moved R3 32.3 mm to (122.5, 73.7), turned to -90 degrees
- moved R9 31.6 mm to (149.1, 69.4), turned to 90 degrees
- moved H4 31.2 mm to (153.9, 97.9)
- moved Q4 30.7 mm to (147.9, 73.6), turned to -90 degrees
- moved R6 23.0 mm to (149.5, 84.1), turned to 90 degrees
- moved H1 22.9 mm to (117.9, 62.1)
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Connections:
- J2 pad 2: Net-(D1-Pad2) -> Net-(D1-A)
- J3 pad 2: Net-(D1-Pad2) -> Net-(D2-A)
- J4 pad 2: Net-(D1-Pad2) -> Net-(D4-A)
- J5 pad 2: Net-(D2-Pad2) -> Net-(D5-A)
- Q1 pad 5: Net-(D1-Pad2) -> Net-(D1-A)
- Q2 pad 5: Net-(D2-Pad2) -> Net-(D2-A)
- Q4 pad 4: /FAN4_BPS -> /FAN3_BPS
- Q4 pad 5: Net-(D4-Pad2) -> Net-(D4-A)
- R3 pad 1: +12V -> /FAN1_BPS
- R3 pad 2: /FAN2_BPS -> GNDPWR
- R5 pad 2: /FAN4_BPS -> /FAN2_BPS
- R6 pad 1: /FAN1_BPS -> /FAN2_BPS
- R7 pad 1: /FAN2_BPS -> +12V
- R7 pad 2: GNDPWR -> /FAN3_BPS
- R9 pad 1: /FAN4_BPS -> /FAN3_BPS
Routing:
- net Net-(D4-Pad2): track 46.2 -> 0.00 mm
- net Net-(D2-Pad2): track 46.2 -> 0.00 mm
- net Net-(D1-Pad2): track 46.2 -> 0.00 mm
- net Net-(D3-Pad2): track 45.9 -> 0.00 mm
- net /FAN4_BPS: track 44.9 -> 0.00 mm
- net /FAN1_BPS: track 34.6 -> 0.00 mm
- net /FAN3_BPS: track 27.3 -> 0.00 mm
- net GNDPWR: track 19.1 -> 0.00 mm, vias 9 -> 0
- net /FAN2_BPS: track 18.6 -> 0.00 mm
- net Net-(LED1-K): track 2.16 -> 0.00 mm
- removed copper zone on F.Cu, net +12V
- removed copper zone on B.Cu, net GNDPWR
Other:
- board size 57.3 x 82.1 mm -> 43.6 x 43.4 mm
- board text removed: "+"
- board text removed: "-"
- board text removed: "12V"
- board text removed: "FAN1"
- board text removed: "FAN2"
- board text removed: "FAN3"
- board text removed: "FAN4"
- board text removed: "LDRBRDConn"
- board text removed: "PWRGND"
- board text removed: "Tasnia was here"
- board text removed: "UTSVT - BPS Fan Board v2.0 Fall 2022"

Commit message: ooga booga
Parts:
- moved J1 15.4 mm to (139.3, 64.5)
Other:
- board size 43.6 x 43.4 mm -> 43.6 x 42.8 mm
Changed lines of the file:
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@@
 		)
 		(fp_text user "${REFERENCE}"
-			(at 0 0 360)
+			(at 0 0 0)
 			(layer "F.Fab")
 			(effects
@@
 		)
 		(fp_text user "${REFERENCE}"
-			(at 0 0 360)
+			(at 0 0 0)
 			(layer "F.Fab")
 			(effects
@@
 		)
 		(fp_text user "${REFERENCE}"
-			(at 0 0 360)
+			(at 0 0 0)
 			(layer "F.Fab")
 			(effects
@@
 		)
 		(fp_text user "${REFERENCE}"
-			(at 0 0 360)
+			(at 0 0 0)
 			(layer "F.Fab")
 			(effects
@@
 	(footprint "Connector_Molex:Molex_Micro-Fit_3.0_43045-0612_2x03_P3.00mm_Vertical"
 		(layer "F.Cu")
-		(at 139.296762 79.92061 180)
+		(at 139.296762 64.52061 180)
 		(descr "Molex Micro-Fit 3.0 Connector System, 43045-0612 (compatible alternatives: 43045-0613, 43045-0624), 3 Pins per row (http://www.molex.com/pdm_docs/sd/430450212_sd.pdf), generated with kicad-footprint-generator")
 		(tags "connector Molex Micro-Fit_3.0 vertical")
 		(property "Reference" "J1"
-			(at 3 -3.67 360)
+			(at 3 -3.67 0)
 			(layer "F.SilkS")
 			(effects
@@
 		)
 		(property "Value" "LDRBRDConn"
-			(at 3 7.51 360)
+			(at 3 7.51 0)
 			(layer "F.Fab")
 			(effects
@@
 		)
 		(fp_text user "${REFERENCE}"
-			(at 3 4.2 360)
+			(at 3 4.2 0)
 			(layer "F.Fab")
 			(effects
@@
 	(gr_rect
 		(start 114.296762 58.52061)
-		(end 157.896762 101.92061)
+		(end 157.896762 101.32061)
 		(stroke
 			(width 0.05)

Commit message: layout go brrr
Parts:
- removed Q1, Q2, Q4, Q5: BUK9M23-80E, Package_TO_SOT_SMD:LFPAK33
- added D1: VSSAF522-M3/H, UTSVT_Passive:DO-221AC, B.Cu at (144.2, 91.5)
- added D2: VSSAF522-M3/H, UTSVT_Passive:DO-221AC, B.Cu at (131.5, 76.8)
- added D4: VSSAF522-M3/H, UTSVT_Passive:DO-221AC, B.Cu at (144.2, 76.6)
- added D5: VSSAF522-M3/H, UTSVT_Passive:DO-221AC, B.Cu at (131.3, 91.6)
- added Q3: IRLML0030, Package_TO_SOT_SMD:SOT-23, B.Cu at (146.7, 97.0)
- added Q6: IRLML0030, Package_TO_SOT_SMD:SOT-23, B.Cu at (134.0, 82.3)
- added Q7: IRLML0030, Package_TO_SOT_SMD:SOT-23, B.Cu at (146.7, 82.2)
- added Q8: IRLML0030, Package_TO_SOT_SMD:SOT-23, B.Cu at (133.8, 97.1)
- LOGO1, R10, R11, R2, R3, R5, R6, R7, R9: moved to B.Cu
- moved LOGO1 79.4 mm to (171.2, 78.5), turned to 180 degrees
- moved LED1 70.8 mm to (153.8, 67.1), turned to 90 degrees
- moved R1 65.5 mm to (153.8, 71.2), turned to -90 degrees
- moved R3 31.6 mm to (143.8, 97.1), turned to 90 degrees
- moved R2 28.9 mm to (141.7, 97.0), turned to -90 degrees
- moved J2 28.2 mm to (142.5, 87.7), turned to 0 degrees
- moved J3 26.5 mm to (129.8, 72.9), turned to 0 degrees
- moved R6 18.4 mm to (131.1, 82.3)
- moved R5 18.3 mm to (129.0, 82.3)
- moved R9 13.8 mm to (143.8, 82.2)
- moved R7 13.7 mm to (141.7, 82.2)
- moved R11 12.7 mm to (130.8, 97.2), turned to 90 degrees
- moved J5 11.7 mm to (129.6, 87.8), turned to 0 degrees
- moved J4 11.5 mm to (142.5, 72.8), turned to 0 degrees
- moved R10 10.3 mm to (128.8, 97.1), turned to -90 degrees
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Connections:
- J2 pad 2: Net-(D1-A) -> /Driver1/FAN-
- J3 pad 2: Net-(D2-A) -> /Driver2/FAN-
- J4 pad 2: Net-(D4-A) -> /Driver3/FAN-
- J5 pad 2: Net-(D5-A) -> /Driver4/FAN-
Routing:
- net +12V: track 0.00 -> 13.8 mm
- net /FAN4_BPS: track 0.00 -> 4.04 mm
- net /FAN2_BPS: track 0.00 -> 4.04 mm
- net /FAN1_BPS: track 0.00 -> 4.04 mm
- net /FAN3_BPS: track 0.00 -> 4.04 mm
- net Net-(LED1-K): track 0.00 -> 2.25 mm
- net GNDPWR: vias 0 -> 4
- added copper zone on B.Cu, net +12V
- added copper zone on B.Cu, net /Driver1/FAN-
- added copper zone on B.Cu, net /Driver2/FAN-
- added copper zone on B.Cu, net /Driver3/FAN-
- added copper zone on B.Cu, net /Driver4/FAN-
- added copper zone on B.Cu, net GNDPWR
- added copper zone on F.Cu, net GNDPWR
Other:
- board size 43.6 x 42.8 mm -> 34.3 x 41.2 mm

Commit message: skibbidi toilet
Parts:
- LOGO1: footprint UTSVT_Special:Hallock_Image_Small -> UTSVT_Special:Hallock_Image_Tiny
- moved LOGO2 47.6 mm to (137.4, 95.6)
- moved LOGO1 34.7 mm to (138.6, 66.7)
- moved J1 1.03 mm to (140.9, 63.0)
- moved LED1 0.95 mm to (152.9, 67.1)
- moved R1 0.95 mm to (152.9, 71.2)
- moved D1 0.25 mm to (144.2, 91.3)
- moved Q3 0.25 mm to (146.7, 96.8)
- moved Q8 0.25 mm to (133.8, 96.9)
- moved R10 0.25 mm to (128.8, 96.9)
- moved R2 0.25 mm to (141.7, 96.8)
- moved R3 0.25 mm to (143.8, 96.8)
- moved D5 0.25 mm to (131.3, 91.4)
- moved J5 0.25 mm to (129.6, 87.5)
- moved R11 0.25 mm to (130.8, 96.9)
- moved J3 0.24 mm to (129.6, 72.8)
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Routing:
- net /FAN4_BPS: track 4.04 -> 47.4 mm
- net /FAN1_BPS: track 4.04 -> 44.0 mm
- net /FAN3_BPS: track 4.04 -> 32.7 mm
- net /FAN2_BPS: track 4.04 -> 29.2 mm
- net +12V: track 13.8 -> 13.3 mm
- added copper zone on F.Cu, net +12V
Other:
- board text added: "+"
- board text added: "-"
- board text added: "FAN 1"
- board text added: "FAN 2"
- board text added: "FAN 3"
- board text added: "FAN 4"
- board text added: "Fan Board Day - Fixed Fall 2024"
- board text added: "Lakshay was here"

Commit message: skibbidi fan
Parts:
- added R12: 100k, Resistor_SMD:R_0805_2012Metric, B.Cu at (144.1, 94.1)
- added R13: 100k, Resistor_SMD:R_0805_2012Metric, B.Cu at (131.9, 94.0)
- added R4: 100k, Resistor_SMD:R_0805_2012Metric, B.Cu at (131.4, 79.4)
- added R8: 100k, Resistor_SMD:R_0805_2012Metric, B.Cu at (143.1, 79.2)
- moved R3 22.5 mm to (129.6, 79.4), turned to -90 degrees
- moved R2 22.2 mm to (127.9, 79.4)
- moved Q3 21.3 mm to (134.1, 79.5)
- moved J2 21.2 mm to (128.9, 71.3)
- moved D1 20.9 mm to (130.1, 75.9)
- moved D4 14.0 mm to (142.9, 90.6)
- moved J4 13.2 mm to (141.6, 86.0)
- moved Q6 12.4 mm to (145.9, 79.4)
- moved Q7 12.1 mm to (146.9, 94.2)
- moved R7 12.0 mm to (140.6, 94.1)
- moved R9 12.0 mm to (142.4, 94.1), turned to -90 degrees
- moved R5 11.2 mm to (139.6, 79.2)
- moved J3 11.1 mm to (140.6, 71.2)
- moved R6 10.9 mm to (141.4, 79.2), turned to -90 degrees
- moved D2 10.6 mm to (141.9, 75.7)
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Connections:
- Q3 pad 1: /FAN1_BPS -> Net-(Q3-G)
- Q6 pad 1: /FAN2_BPS -> Net-(Q6-G)
- Q7 pad 1: /FAN3_BPS -> Net-(Q7-G)
- Q8 pad 1: /FAN4_BPS -> Net-(Q8-G)
- R11 pad 1: /FAN4_BPS -> GNDPWR
- R11 pad 2: GNDPWR -> /FAN4_BPS
- R3 pad 1: /FAN1_BPS -> GNDPWR
- R3 pad 2: GNDPWR -> /FAN1_BPS
- R6 pad 1: /FAN2_BPS -> GNDPWR
- R6 pad 2: GNDPWR -> /FAN2_BPS
- R9 pad 1: /FAN3_BPS -> GNDPWR
- R9 pad 2: GNDPWR -> /FAN3_BPS
Routing:
- net /FAN4_BPS: track 47.4 -> 3.50 mm
- net /FAN1_BPS: track 44.0 -> 3.50 mm
- net /FAN3_BPS: track 32.7 -> 3.50 mm
- net /FAN2_BPS: track 29.2 -> 3.50 mm
- net Net-(Q7-G): track 0.00 -> 2.76 mm
- net Net-(Q8-G): track 0.00 -> 2.76 mm
- net Net-(Q6-G): track 0.00 -> 2.76 mm
- net Net-(Q3-G): track 0.00 -> 2.76 mm
Other:
- board text removed: "FAN 1"
- board text removed: "FAN 2"
- board text removed: "FAN 3"

Commit message: done
Parts:
- moved Q6 20.2 mm to (133.1, 95.1)
- moved D2 19.7 mm to (130.3, 91.6)
- moved R5 19.6 mm to (128.1, 95.1)
- moved R6 19.4 mm to (130.2, 95.1)
- moved J3 18.7 mm to (130.4, 86.8)
- moved R4 17.5 mm to (148.9, 80.3), turned to -90 degrees
- moved R8 17.3 mm to (136.1, 95.1), turned to -90 degrees
- moved R13 14.3 mm to (136.1, 80.3), turned to -90 degrees
- moved J2 14.2 mm to (143.1, 72.1)
- moved J5 13.9 mm to (130.4, 72.1)
- moved Q8 13.9 mm to (133.1, 80.3)
- moved R10 13.7 mm to (128.1, 80.3)
- moved R11 13.7 mm to (130.2, 80.3)
- moved D5 13.6 mm to (130.3, 76.9)
- moved R3 13.3 mm to (142.9, 80.3)
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Connections:
- R10 pad 2: /FAN4_BPS -> Net-(Q8-G)
- R11 pad 2: /FAN4_BPS -> Net-(Q8-G)
- R2 pad 2: /FAN1_BPS -> Net-(Q3-G)
- R3 pad 2: /FAN1_BPS -> Net-(Q3-G)
- R5 pad 2: /FAN2_BPS -> Net-(Q6-G)
- R6 pad 2: /FAN2_BPS -> Net-(Q6-G)
- R7 pad 2: /FAN3_BPS -> Net-(Q7-G)
- R9 pad 2: /FAN3_BPS -> Net-(Q7-G)
Routing:
- net /FAN3_BPS: track 3.50 -> 51.0 mm, vias 0 -> 2
- net /FAN1_BPS: track 3.50 -> 35.5 mm, vias 0 -> 2
- net /FAN2_BPS: track 3.50 -> 33.0 mm
- net /FAN4_BPS: track 3.50 -> 22.3 mm
- net Net-(Q7-G): track 2.76 -> 12.6 mm
- net Net-(Q6-G): track 2.76 -> 8.90 mm
- net Net-(Q8-G): track 2.76 -> 8.90 mm
- net Net-(Q3-G): track 2.76 -> 8.64 mm
- net GNDPWR: vias 4 -> 6
Other:
- board text added: "Fan 1 + -"
- board text added: "Fan 2 + -"
- board text added: "Fan 3 + -"
- board text added: "Fan 4 + -"
- board text removed: "FAN 4"
