File: BPS-Fan.kicad_sch (KiCad schematic)
At the start: 37 parts, among them J1 LDRBRDConn, J10 FAN9, J11 FAN10, J12 FAN11, J13 FAN12, J2 FAN1, J3 FAN2, J4 FAN3, J5 FAN4, J6 FAN5, J7 FAN6, J8 FAN7, J9 FAN8, Q1 BUK9M23-80E, Q2 BUK9M23-80E, Q3 BUK9M23-80E, Q4 BUK9M23-80E

Commit message: fan go brrr
Parts:
- removed D1, D2, D3, D4: V2F22HM, UTSVT_Passive:V2F22HM, symbol Diode:C3D25170H
- removed J10: FAN9, UTSVT_Connectors:Molex_MicroFit3.0_1x2xP3.00mm_PolarizingPeg_Vertical, symbol Connector_Generic:Conn_01x02
- removed J11: FAN10, UTSVT_Connectors:Molex_MicroFit3.0_1x2xP3.00mm_PolarizingPeg_Vertical, symbol Connector_Generic:Conn_01x02
- removed J12: FAN11, UTSVT_Connectors:Molex_MicroFit3.0_1x2xP3.00mm_PolarizingPeg_Vertical, symbol Connector_Generic:Conn_01x02
- removed J13: FAN12, UTSVT_Connectors:Molex_MicroFit3.0_1x2xP3.00mm_PolarizingPeg_Vertical, symbol Connector_Generic:Conn_01x02
- removed J2: FAN1, UTSVT_Connectors:Molex_MicroFit3.0_1x2xP3.00mm_PolarizingPeg_Vertical, symbol Connector_Generic:Conn_01x02
- removed J3: FAN2, UTSVT_Connectors:Molex_MicroFit3.0_1x2xP3.00mm_PolarizingPeg_Vertical, symbol Connector_Generic:Conn_01x02
- removed J4: FAN3, UTSVT_Connectors:Molex_MicroFit3.0_1x2xP3.00mm_PolarizingPeg_Vertical, symbol Connector_Generic:Conn_01x02
- removed J5: FAN4, UTSVT_Connectors:Molex_MicroFit3.0_1x2xP3.00mm_PolarizingPeg_Vertical, symbol Connector_Generic:Conn_01x02
- removed J6: FAN5, UTSVT_Connectors:Molex_MicroFit3.0_1x2xP3.00mm_PolarizingPeg_Vertical, symbol Connector_Generic:Conn_01x02
- removed J7: FAN6, UTSVT_Connectors:Molex_MicroFit3.0_1x2xP3.00mm_PolarizingPeg_Vertical, symbol Connector_Generic:Conn_01x02
- removed J8: FAN7, UTSVT_Connectors:Molex_MicroFit3.0_1x2xP3.00mm_PolarizingPeg_Vertical, symbol Connector_Generic:Conn_01x02
- removed J9: FAN8, UTSVT_Connectors:Molex_MicroFit3.0_1x2xP3.00mm_PolarizingPeg_Vertical, symbol Connector_Generic:Conn_01x02
- removed Q1, Q2, Q3, Q4: BUK9M23-80E, Package_TO_SOT_SMD:LFPAK33, symbol Transistor_FET:BUK9M23-80EX
- removed R2, R3, R4, R5, R6, R7, R8, R9: 100k, Resistor_SMD:R_0805_2012Metric, symbol Device:R
Other:
- added sheet Driver (driver.kicad_sch)
- added sheet Driver1 (driver.kicad_sch)
- added sheet Driver2 (driver.kicad_sch)
- added sheet Driver3 (driver.kicad_sch)
- moved on the sheet: LED1, R1

Commit message: layout go brrr
Other:
- removed sheet Driver
- added sheet Driver4 (driver.kicad_sch)
Changed lines of the file:
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@@
 			)
 		)
-		(property "Description" ""
+		(property "Description" "Mounting Hole without connection"
 			(at 245.11 57.15 0)
 			(effects
@@
 			)
 		)
-		(property "Description" ""
+		(property "Description" "Mounting Hole without connection"
 			(at 245.11 64.77 0)
 			(effects
@@
 			)
 		)
-		(property "Description" ""
+		(property "Description" "Mounting Hole without connection"
 			(at 245.11 72.39 0)
 			(effects
@@
 			)
 		)
-		(property "Description" ""
+		(property "Description" "Mounting Hole without connection"
 			(at 245.11 81.28 0)
 			(effects
@@
 			)
 		)
-		(property "Datasheet" "https://www.mouser.com/ProductDetail/71-CRCW080510K0FKEAC"
+		(property "Datasheet" "~"
 			(at 165.1 77.47 0)
 			(effects
@@
 			)
 		)
-		(property "Description" ""
+		(property "Description" "Resistor"
 			(at 165.1 77.47 0)
 			(effects
@@
 			)
 		)
-		(property "Datasheet" "https://www.mouser.com/datasheet/2/216/APTD2012LVBC-D-1101043.pdf"
+		(property "Datasheet" "~"
 			(at 165.1 69.85 0)
 			(effects
@@
 			)
 		)
-		(property "Description" ""
+		(property "Description" "Light emitting diode"
 			(at 165.1 69.85 0)
 			(effects
@@
 			)
 		)
-		(property "Description" ""
+		(property "Description" "Power symbol creates a global label with name \"+12V\""
 			(at 165.1 66.04 0)
 			(effects
@@
 			)
 		)
-		(property "Description" ""
+		(property "Description" "Power symbol creates a global label with name \"GNDPWR\" , global ground"
 			(at 165.1 81.28 0)
 			(effects
@@
 			)
 		)
-		(property "Description" ""
+		(property "Description" "Graph footprint placeholder"
 			(at 269.24 58.42 0)
 			(effects
@@
 			)
 		)
-		(property "Description" ""
+		(property "Description" "Graph footprint placeholder"
 			(at 269.24 66.04 0)
 			(effects
@@
 			)
 		)
-		(property "Description" ""
+		(property "Description" "Power symbol creates a global label with name \"+12V\""
 			(at 62.23 63.5 0)
 			(effects
@@
 			)
 		)
-		(property "Description" ""
+		(property "Description" "Power symbol creates a global label with name \"GNDPWR\" , global ground"
 			(at 41.91 71.12 0)
 			(effects
@@
 			)
 		)
-		(property "Datasheet" "https://www.mouser.com/datasheet/2/276/3/0430450626_PCB_HEADERS-2832587.pdf"
+		(property "Datasheet" "~"
 			(at 50.8 66.04 0)
 			(effects
@@
 			)
 		)
-		(property "Description" ""
+		(property "Description" "Generic connector, double row, 02x03, top/bottom pin numbering scheme (row 1: 1...pins_per_row, row2: pins_per_row+1 ... num_pins), script generated (kicad-library-utils/schlib/autogen/connector/)"
 			(at 50.8 66.04 0)
 			(effects
@@
 			(color 0 0 0 0.0000)
 		)
-		(property "Sheetname" "Driver"
+		(property "Sheetname" "Driver1"
 			(at 96.52 62.7884 0)
 			(effects
@@
 			(color 0 0 0 0.0000)
 		)
-		(property "Sheetname" "Driver2"
+		(property "Sheetname" "Driver3"
 			(at 96.52 91.9984 0)
 			(effects
@@
 			(color 0 0 0 0.0000)
 		)
-		(property "Sheetname" "Driver1"
+		(property "Sheetname" "Driver2"
 			(at 96.52 78.0284 0)
 			(effects
@@
 			(color 0 0 0 0.0000)
 		)
-		(property "Sheetname" "Driver3"
+		(property "Sheetname" "Driver4"
 			(at 96.52 105.9684 0)
 			(effects

Commit message: skibbidi toilet
Parts:
- LOGO1: footprint UTSVT_Special:Hallock_Image_Small -> UTSVT_Special:Hallock_Image_Tiny
Changed lines of the file:
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@@
 			)
 		)
-		(property "Footprint" "UTSVT_Special:Hallock_Image_Small"
+		(property "Footprint" "UTSVT_Special:Hallock_Image_Tiny"
 			(at 269.24 56.515 0)
 			(effects
