File: driver.kicad_sch (KiCad schematic)
At the start: 5 parts, among them J2 FAN7, Q1 BUK9M23-80E

Commit message: layout go brrr
Parts:
- removed Q1: BUK9M23-80E, Package_TO_SOT_SMD:LFPAK33, symbol Transistor_FET:BUK9M23-80EX
- added Q3: IRLML0030, Package_TO_SOT_SMD:SOT-23, symbol Transistor_FET:IRLML0030
- D1: value V2F22HM -> VSSAF522-M3/H; footprint UTSVT_Passive:V2F22HM -> UTSVT_Passive:DO-221AC
Connections:
- net GNDPWR: now also Q3.2 (S)
- net PWM: now also Q3.1 (G)
- net FAN-: now reaches D1.2 (A), J2.2 (Pin_2)
- net FAN-: now also Q3.3 (D)
Other:
- moved on the sheet: J2
Changed lines of the file:
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@@
 	(wire
 		(pts
-			(xy 147.32 82.55) (xy 156.21 82.55)
+			(xy 147.32 82.55) (xy 160.02 82.55)
 		)
 		(stroke
@@
 	(wire
 		(pts
-			(xy 156.21 80.01) (xy 153.67 80.01)
-		)
-		(stroke
-			(width 0)
-			(type default)
+			(xy 160.02 80.01) (xy 153.67 80.01)
+		)
+		(stroke
+			(width 0)
+			(type default)
+		)
+	)
+	(label "FAN-"
+		(at 153.67 82.55 0)
+		(fields_autoplaced yes)
+		(effects
+			(font
+				(size 1.27 1.27)
+			)
+			(justify left bottom)
 		)
 	)
@@
 			)
 		)
-		(property "Datasheet" "https://www.mouser.com/ProductDetail/Vishay-Dale/CRCW0805100KFKEAC?qs=sGAEpiMZZMvdGkrng054t0DrEhLhGh8gZRT9GjFuHWDV3jEqj5sSqw%3D%3D"
+		(property "Datasheet" "~"
 			(at 127 82.55 0)
 			(effects
@@
 			)
 		)
-		(property "Description" ""
+		(property "Description" "Resistor"
 			(at 127 82.55 0)
 			(effects
@@
 			)
 		)
-		(property "Value" "V2F22HM"
-			(at 135.89 81.28 90)
-			(effects
-				(font
-					(size 1.27 1.27)
-				)
-				(justify left)
-			)
-		)
-		(property "Footprint" "UTSVT_Passive:V2F22HM"
+		(property "Value" "VSSAF522-M3/H"
+			(at 129.794 76.708 90)
+			(effects
+				(font
+					(size 1.27 1.27)
+				)
+				(justify left)
+			)
+		)
+		(property "Footprint" "UTSVT_Passive:DO-221AC"
 			(at 142.875 78.74 0)
 			(effects
@@
 			)
 		)
-		(property "Datasheet" "https://www.mouser.com/datasheet/2/427/v2f22-1767661.pdf"
+		(property "Datasheet" "https://www.mouser.com/ProductDetail/Vishay-General-Semiconductor/VSSAF522-M3-H?qs=UkDUCjYnTB00gpgD%2Fb%2Fw%252BA%3D%3D"
 			(at 147.32 78.74 0)
 			(effects
@@
 			)
 		)
-		(property "Description" ""
+		(property "Description" "Power symbol creates a global label with name \"GNDPWR\" , global ground"
 			(at 147.32 101.6 0)
 			(effects
@@
 	(symbol
 		(lib_id "Connector_Generic:Conn_01x02")
-		(at 161.29 80.01 0)
+		(at 165.1 80.01 0)
 		(unit 1)
 		(exclude_from_sim no)
@@
 		(dnp no)
 		(property "Reference" "J2"
-			(at 163.322 80.2132 0)
+			(at 167.132 80.2132 0)
 			(effects
 				(font
@@
 		)
 		(property "Value" "FAN7"
-			(at 163.322 82.5246 0)
+			(at 167.132 82.5246 0)
 			(effects
 				(font
@@
 		)
 		(property "Footprint" "UTSVT_Connectors:Molex_MicroFit3.0_1x2xP3.00mm_PolarizingPeg_Vertical"
-			(at 161.29 80.01 0)
-			(effects
-				(font
-					(size 1.27 1.27)
-				)
-				(hide yes)
-			)
-		)
-		(property "Datasheet" "https://www.mouser.com/datasheet/2/276/3/0436500226_PCB_HEADERS-2845455.pdf"
-			(at 161.29 80.01 0)
-			(effects
-				(font
-					(size 1.27 1.27)
-				)
-				(hide yes)
-			)
-		)
-		(property "Description" ""
-			(at 161.29 80.01 0)
+			(at 165.1 80.01 0)
+			(effects
+				(font
+					(size 1.27 1.27)
+				)
+				(hide yes)
+			)
+		)
+		(property "Datasheet" "~"
+			(at 165.1 80.01 0)
+			(effects
+				(font
+					(size 1.27 1.27)
+				)
+				(hide yes)
+			)
+		)
+		(property "Description" "Generic connector, single row, 01x02, script generated (kicad-library-utils/schlib/autogen/connector/)"
+			(at 165.1 80.01 0)
 			(effects
 				(font
@@
 				(path "/e60847d4-a954-40b9-b9c4-54b73957661c/6eaa0a11-7e18-4b05-9cbf-a4206d1f64dd"
 					(reference "J5")
-					(unit 1)
-				)
-			)
-		)
-	)
-	(symbol
-		(lib_id "Transistor_FET:BUK9M23-80EX")
-		(at 144.78 90.17 0)
-		(unit 1)
-		(exclude_from_sim no)
-		(in_bom yes)
-		(on_board yes)
-		(dnp no)
-		(property "Reference" "Q1"
-			(at 149.9616 89.0016 0)
-			(effects
-				(font
-					(size 1.27 1.27)
-				)
-				(justify left)
-			)
-		)
-		(property "Value" "BUK9M23-80E"
-			(at 151.13 96.52 0)
-			(effects
-				(font
-					(size 1.27 1.27)
-				)
-				(justify left)
-			)
-		)
-		(property "Footprint" "Package_TO_SOT_SMD:LFPAK33"
-			(at 149.86 92.075 0)
-			(effects
-				(font
-					(size 1.27 1.27)
-					(italic yes)
-				)
-				(justify left)
-				(hide yes)
-			)
-		)
-		(property "Datasheet" "https://assets.nexperia.com/documents/data-sheet/BUK9M23-80E.pdf"
-			(at 144.78 90.17 90)
-			(effects
-				(font
-					(size 1.27 1.27)
-				)
-				(justify left)
-				(hide yes)
-			)
-		)
-		(property "Description" ""
-			(at 144.78 90.17 0)
-			(effects
-				(font
-					(size 1.27 1.27)
-				)
-				(hide yes)
-			)
-		)
-		(pin "1"
-		)
-		(pin "2"
-		)
-		(pin "3"
-		)
-		(pin "4"
-		)
-		(pin "5"
-		)
-		(instances
-			(project "BPS-Fan"
-				(path "/e60847d4-a954-40b9-b9c4-54b73957661c/105d6206-78eb-4194-afd4-8d8c1c7531a1"
-					(reference "Q1")
-					(unit 1)
-				)
-				(path "/e60847d4-a954-40b9-b9c4-54b73957661c/324616d9-bf64-418c-88ee-8b9e8f32727d"
-					(reference "Q4")
-					(unit 1)
-				)
-				(path "/e60847d4-a954-40b9-b9c4-54b73957661c/48a070bc-ea68-4415-9c4a-a4a1af37f712"
-					(reference "Q2")
-					(unit 1)
-				)
-				(path "/e60847d4-a954-40b9-b9c4-54b73957661c/6eaa0a11-7e18-4b05-9cbf-a4206d1f64dd"
-					(reference "Q5")
 					(unit 1)
 				)
@@
 			)
 		)
-		(property "Description" ""
+		(property "Description" "Power symbol creates a global label with name \"+12V\""
 			(at 147.32 71.12 0)
 			(effects
@@
 				(path "/e60847d4-a954-40b9-b9c4-54b73957661c/6eaa0a11-7e18-4b05-9cbf-a4206d1f64dd"
 					(reference "#PWR010")
+					(unit 1)
+				)
+			)
+		)
+	)
+	(symbol
+		(lib_id "Transistor_FET:IRLML0030")
+		(at 144.78 90.17 0)
+		(unit 1)
+		(exclude_from_sim no)
+		(in_bom yes)
+		(on_board yes)
+		(dnp no)
+		(fields_autoplaced yes)
+		(property "Reference" "Q3"
+			(at 151.13 88.8999 0)
+			(effects
+				(font
+					(size 1.27 1.27)
+				)
+				(justify left)
+			)
+		)
+		(property "Value" "IRLML0030"
+			(at 151.13 91.4399 0)
+			(effects
+				(font
+					(size 1.27 1.27)
+				)
+				(justify left)
+			)
+		)
+		(property "Footprint" "Package_TO_SOT_SMD:SOT-23"
+			(at 149.86 92.075 0)
+			(effects
+				(font
+					(size 1.27 1.27)
+					(italic yes)
+				)
+				(justify left)
+				(hide yes)
+			)
+		)
+		(property "Datasheet" "https://www.infineon.com/dgdl/irlml0030pbf.pdf?fileId=5546d462533600a401535664773825df"
+			(at 149.86 93.98 0)
+			(effects
+				(font
+					(size 1.27 1.27)
+				)
+				(justify left)
+				(hide yes)
+			)
+		)
+		(property "Description" "5.3A Id, 30V Vds, 27mOhm Rds, N-Channel HEXFET Power MOSFET, SOT-23"
+			(at 144.78 90.17 0)
+			(effects
+				(font
+					(size 1.27 1.27)
+				)
+				(hide yes)
+			)
+		)
+		(pin "3"
+		)
+		(pin "1"
+		)
+		(pin "2"
+		)
+		(instances
+			(project ""
+				(path "/e60847d4-a954-40b9-b9c4-54b73957661c/105d6206-78eb-4194-afd4-8d8c1c7531a1"
+					(reference "Q3")
+					(unit 1)
+				)
+				(path "/e60847d4-a954-40b9-b9c4-54b73957661c/324616d9-bf64-418c-88ee-8b9e8f32727d"
+					(reference "Q7")
+					(unit 1)
+				)
+				(path "/e60847d4-a954-40b9-b9c4-54b73957661c/48a070bc-ea68-4415-9c4a-a4a1af37f712"
+					(reference "Q6")
+					(unit 1)
+				)
+				(path "/e60847d4-a954-40b9-b9c4-54b73957661c/6eaa0a11-7e18-4b05-9cbf-a4206d1f64dd"
+					(reference "Q8")
 					(unit 1)
 				)
@@
 			)
 		)
-		(property "Datasheet" "https://www.mouser.com/ProductDetail/Vishay-Dale/CRCW0805100KFKEAC?qs=sGAEpiMZZMvdGkrng054t0DrEhLhGh8gZRT9GjFuHWDV3jEqj5sSqw%3D%3D"
+		(property "Datasheet" "~"
 			(at 135.89 97.79 0)
 			(effects
@@
 			)
 		)
-		(property "Description" ""
+		(property "Description" "Resistor"
 			(at 135.89 97.79 0)
 			(effects

Commit message: skibbidi fan
Parts:
- added R4: 100k, Resistor_SMD:R_0805_2012Metric, symbol Device:R
Connections:
- net GNDPWR: now also R3.1; no longer R3.2
- net PWM: now also R3.2, R4.1; no longer Q3.1 (G), R3.1
- new net: Q3.1 (G), R4.2
Other:
- note added: "current limiting resistor on gate Only solder pullup or pulldown resistor (NOT BOTH)"
- moved on the sheet: Q3, R2, R3

Commit message: done
Connections:
- net PWM: no longer R2.2, R3.2
- net at Q3.1 (G), R4.2: now also R2.2, R3.2
Other:
- moved on the sheet: R2, R3
